File: carteCMS/cms-KiCad/accordeur_analog.kicad_sch (KiCad schematic)
At the start: 18 parts, among them U1 LM358, U2 max7426cua+T, U4 CD4093BM96

Commit message: v2 - schéma et empruntes terminés (normalement)
Parts:
- removed U1: LM358, accordeurEmp:LM358emp, symbol Amplifier_Operational:LM358
- removed U2: max7426cua+T, 21-0036K_MXM, symbol 2026-09-04_07-21-49:max7426cua+T
- removed U4: CD4093BM96, D14, symbol 2026-09-04_07-53-46:CD4093BM96
- added IC1: CD4093BM, Package_SO:SO-14_5.3x10.2mm_P1.27mm, symbol accordeurSym:CD4093BM
- added U1: LM358, Package_TO_SOT_SMD:SOT-353_SC-70-5, symbol Amplifier_Operational:TLV172IDCK
- added U3: max7426cua+T, accordeurEmp:MAX7426, symbol accordeurSym:max7426cua+T
- C10, C11, C9: footprint (none) -> Capacitor_SMD:C_0805_2012Metric
- MK1: footprint (none) -> accordeurEmp:micro-KECG2740PBJ
- TP1, TP2, TP3, TP4: footprint (none) -> TestPoint:TestPoint_Pad_D2.0mm
Connections:
- net +5V: now also IC1.14 (VDD), U1.5 (V+), U3.4 (VDD), U3.7 (*SHDN)
- net 100xFc: now also U3.1 (COM), U3.6 (OS), U3.8 (CLK)
- net Fmesure: now also IC1.11 (M)
- net GND: now also IC1.7 (VSS), U1.2 (V-), U3.3 (GND)
- net at R6.2, TP1.1: now also U1.4, U3.2 (IN)
- net at TP3.1: now also IC1.12 (G), IC1.13 (H), U3.5 (OUT)
- net at R4.2, R5.1: now also U1.1 (+)
- net at R3.2, R6.1: now also U1.3 (-)
- no-connect marks 12 -> 9

Commit message: Début routage (avant pistes)
Connections:
- net 100xFc: no longer C4.2, U3.1 (COM), U3.6 (OS)
- new net: C4.2, U3.1 (COM), U3.6 (OS)
Other:
- moved on the sheet: TP2
Changed lines of the file:
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@@
-	)
-	(junction
-		(at 175.26 101.6)
-		(diameter 0)
-		(color 0 0 0 0)
 	)
 	(junction
@@
 	)
 	(junction
-		(at 175.26 76.2)
-		(diameter 0)
-		(color 0 0 0 0)
-	)
-	(junction
 		(at 243.84 101.6)
 		(diameter 0)
@@
 	)
 	(junction
+		(at 166.37 101.6)
+		(diameter 0)
+		(color 0 0 0 0)
+	)
+	(junction
 		(at 241.3 57.15)
 		(diameter 0)
 		(color 0 0 0 0)
 	)
-	(junction
-		(at 175.26 71.12)
-		(diameter 0)
-		(color 0 0 0 0)
-	)
 	(no_connect
 		(at 207.01 67.31)
@@
 	(wire
 		(pts
-			(xy 175.26 101.6) (xy 175.26 104.14)
+			(xy 166.37 71.12) (xy 166.37 101.6)
 		)
 		(stroke
@@
 	(wire
 		(pts
-			(xy 175.26 71.12) (xy 162.56 71.12)
-		)
-		(stroke
-			(width 0)
-			(type default)
-		)
-	)
-	(wire
-		(pts
 			(xy 125.73 71.12) (xy 125.73 59.69)
 		)
@@
 	(wire
 		(pts
-			(xy 176.53 101.6) (xy 175.26 101.6)
+			(xy 167.64 101.6) (xy 166.37 101.6)
 		)
 		(stroke
@@
 	(wire
 		(pts
+			(xy 162.56 71.12) (xy 166.37 71.12)
+		)
+		(stroke
+			(width 0)
+			(type default)
+		)
+	)
+	(wire
+		(pts
 			(xy 127 59.69) (xy 127 55.88)
 		)
@@
 	(wire
 		(pts
-			(xy 175.26 71.12) (xy 175.26 59.69)
-		)
-		(stroke
-			(width 0)
-			(type default)
-		)
-	)
-	(wire
-		(pts
 			(xy 243.84 64.77) (xy 243.84 101.6)
 		)
@@
 	(wire
 		(pts
-			(xy 175.26 76.2) (xy 175.26 71.12)
+			(xy 166.37 101.6) (xy 166.37 104.14)
+		)
+		(stroke
+			(width 0)
+			(type default)
+		)
+	)
+	(wire
+		(pts
+			(xy 175.26 59.69) (xy 175.26 76.2)
 		)
 		(stroke
@@
 		(pts
 			(xy 162.56 78.74) (xy 181.61 78.74)
-		)
-		(stroke
-			(width 0)
-			(type default)
-		)
-	)
-	(wire
-		(pts
-			(xy 175.26 101.6) (xy 175.26 76.2)
 		)
 		(stroke
@@
 	(hierarchical_label "100xFc"
 		(shape input)
-		(at 175.26 104.14 270)
+		(at 166.37 104.14 270)
 		(fields_autoplaced yes)
 		(effects
@@
 		)
 		(instances
-			(project "projet-KiCad"
+			(project "cms-KiCad"
 				(path "/59f7da0b-cec5-4ac9-8c02-026d0daeaa65/3402a500-47ed-4144-af75-73ef246582be"
 					(reference "C9")
@@
 		)
 		(instances
-			(project "projet-KiCad"
+			(project "cms-KiCad"
 				(path "/59f7da0b-cec5-4ac9-8c02-026d0daeaa65/3402a500-47ed-4144-af75-73ef246582be"
 					(reference "#PWR028")
@@
 		)
 		(instances
-			(project "projet-KiCad"
+			(project "cms-KiCad"
 				(path "/59f7da0b-cec5-4ac9-8c02-026d0daeaa65/3402a500-47ed-4144-af75-73ef246582be"
 					(reference "R5")
@@
 		)
 		(instances
-			(project "projet-KiCad"
+			(project "cms-KiCad"
 				(path "/59f7da0b-cec5-4ac9-8c02-026d0daeaa65/3402a500-47ed-4144-af75-73ef246582be"
 					(reference "#PWR04")
@@
 		)
 		(instances
-			(project "projet-KiCad"
+			(project "cms-KiCad"
 				(path "/59f7da0b-cec5-4ac9-8c02-026d0daeaa65/3402a500-47ed-4144-af75-73ef246582be"
 					(reference "R3")
@@
 		)
 		(instances
-			(project "projet-KiCad"
+			(project "cms-KiCad"
 				(path "/59f7da0b-cec5-4ac9-8c02-026d0daeaa65/3402a500-47ed-4144-af75-73ef246582be"
 					(reference "#PWR013")
@@
 		)
 		(instances
-			(project "projet-KiCad"
+			(project "cms-KiCad"
 				(path "/59f7da0b-cec5-4ac9-8c02-026d0daeaa65/3402a500-47ed-4144-af75-73ef246582be"
 					(reference "C11")
@@
 		)
 		(instances
-			(project ""
+			(project "cms-KiCad"
 				(path "/59f7da0b-cec5-4ac9-8c02-026d0daeaa65/3402a500-47ed-4144-af75-73ef246582be"
 					(reference "IC1")
@@
 		)
 		(instances
-			(project "projet-KiCad"
+			(project "cms-KiCad"
 				(path "/59f7da0b-cec5-4ac9-8c02-026d0daeaa65/3402a500-47ed-4144-af75-73ef246582be"
 					(reference "#PWR07")
@@
 		)
 		(instances
-			(project "projet-KiCad"
+			(project "cms-KiCad"
 				(path "/59f7da0b-cec5-4ac9-8c02-026d0daeaa65/3402a500-47ed-4144-af75-73ef246582be"
 					(reference "R4")
@@
 		)
 		(instances
-			(project "projet-KiCad"
+			(project "cms-KiCad"
 				(path "/59f7da0b-cec5-4ac9-8c02-026d0daeaa65/3402a500-47ed-4144-af75-73ef246582be"
 					(reference "TP4")
@@
 	(symbol
 		(lib_id "Connector:TestPoint")
-		(at 176.53 101.6 270)
+		(at 167.64 101.6 270)
 		(unit 1)
 		(exclude_from_sim no)
@@
 		(fields_autoplaced yes)
 		(property "Reference" "TP2"
-			(at 181.61 100.3299 90)
+			(at 172.72 100.3299 90)
 			(effects
 				(font
@@
 		)
 		(property "Value" "TestPoint"
-			(at 181.61 102.8699 90)
+			(at 172.72 102.8699 90)
 			(effects
 				(font
@@
 		)
 		(property "Footprint" "TestPoint:TestPoint_Pad_D2.0mm"
-			(at 176.53 106.68 0)
+			(at 167.64 106.68 0)
 			(effects
 				(font
@@
 		)
 		(property "Datasheet" "~"
-			(at 176.53 106.68 0)
+			(at 167.64 106.68 0)
 			(effects
 				(font
@@
 		)
 		(property "Description" "test point"
-			(at 176.53 101.6 0)
-			(effects
-				(font
-					(size 1.27 1.27)
-				)
-				(hide yes)
-			)
-		)
-		(pin "1"
-		)
-		(instances
-			(project "projet-KiCad"
+			(at 167.64 101.6 0)
+			(effects
+				(font
+					(size 1.27 1.27)
+				)
+				(hide yes)
+			)
+		)
+		(pin "1"
+		)
+		(instances
+			(project "cms-KiCad"
 				(path "/59f7da0b-cec5-4ac9-8c02-026d0daeaa65/3402a500-47ed-4144-af75-73ef246582be"
 					(reference "TP2")
@@
 		)
 		(instances
-			(project "projet-KiCad"
+			(project "cms-KiCad"
 				(path "/59f7da0b-cec5-4ac9-8c02-026d0daeaa65/3402a500-47ed-4144-af75-73ef246582be"
 					(reference "#PWR011")
@@
 		)
 		(instances
-			(project "projet-KiCad"
+			(project "cms-KiCad"
 				(path "/59f7da0b-cec5-4ac9-8c02-026d0daeaa65/3402a500-47ed-4144-af75-73ef246582be"
 					(reference "R2")
@@
 		)
 		(instances
-			(project "projet-KiCad"
+			(project "cms-KiCad"
 				(path "/59f7da0b-cec5-4ac9-8c02-026d0daeaa65/3402a500-47ed-4144-af75-73ef246582be"
 					(reference "TP3")
@@
 		)
 		(instances
-			(project ""
+			(project "cms-KiCad"
 				(path "/59f7da0b-cec5-4ac9-8c02-026d0daeaa65/3402a500-47ed-4144-af75-73ef246582be"
 					(reference "U1")
@@
 		)
 		(instances
-			(project "projet-KiCad"
+			(project "cms-KiCad"
 				(path "/59f7da0b-cec5-4ac9-8c02-026d0daeaa65/3402a500-47ed-4144-af75-73ef246582be"
 					(reference "#PWR029")
@@
 		)
 		(instances
-			(project "projet-KiCad"
+			(project "cms-KiCad"
 				(path "/59f7da0b-cec5-4ac9-8c02-026d0daeaa65/3402a500-47ed-4144-af75-73ef246582be"
 					(reference "#PWR09")
@@
 		)
 		(instances
-			(project "projet-KiCad"
+			(project "cms-KiCad"
 				(path "/59f7da0b-cec5-4ac9-8c02-026d0daeaa65/3402a500-47ed-4144-af75-73ef246582be"
 					(reference "MK1")
@@
 		)
 		(instances
-			(project "projet-KiCad"
+			(project "cms-KiCad"
 				(path "/59f7da0b-cec5-4ac9-8c02-026d0daeaa65/3402a500-47ed-4144-af75-73ef246582be"
 					(reference "#PWR08")
@@
 		)
 		(instances
-			(project "projet-KiCad"
+			(project "cms-KiCad"
 				(path "/59f7da0b-cec5-4ac9-8c02-026d0daeaa65/3402a500-47ed-4144-af75-73ef246582be"
 					(reference "#PWR03")
@@
 		)
 		(instances
-			(project "projet-KiCad"
+			(project "cms-KiCad"
 				(path "/59f7da0b-cec5-4ac9-8c02-026d0daeaa65/3402a500-47ed-4144-af75-73ef246582be"
 					(reference "#PWR06")
@@
 		)
 		(instances
-			(project ""
+			(project "cms-KiCad"
 				(path "/59f7da0b-cec5-4ac9-8c02-026d0daeaa65/3402a500-47ed-4144-af75-73ef246582be"
 					(reference "U3")
@@
 		)
 		(instances
-			(project "projet-KiCad"
+			(project "cms-KiCad"
 				(path "/59f7da0b-cec5-4ac9-8c02-026d0daeaa65/3402a500-47ed-4144-af75-73ef246582be"
 					(reference "TP1")
@@
 		)
 		(instances
-			(project "projet-KiCad"
+			(project "cms-KiCad"
 				(path "/59f7da0b-cec5-4ac9-8c02-026d0daeaa65/3402a500-47ed-4144-af75-73ef246582be"
 					(reference "#PWR012")
@@
 		)
 		(instances
-			(project "projet-KiCad"
+			(project "cms-KiCad"
 				(path "/59f7da0b-cec5-4ac9-8c02-026d0daeaa65/3402a500-47ed-4144-af75-73ef246582be"
 					(reference "C4")
@@
 		)
 		(instances
-			(project "projet-KiCad"
+			(project "cms-KiCad"
 				(path "/59f7da0b-cec5-4ac9-8c02-026d0daeaa65/3402a500-47ed-4144-af75-73ef246582be"
 					(reference "C2")
@@
 		)
 		(instances
-			(project "projet-KiCad"
+			(project "cms-KiCad"
 				(path "/59f7da0b-cec5-4ac9-8c02-026d0daeaa65/3402a500-47ed-4144-af75-73ef246582be"
 					(reference "#PWR05")
@@
 		)
 		(instances
-			(project "projet-KiCad"
+			(project "cms-KiCad"
 				(path "/59f7da0b-cec5-4ac9-8c02-026d0daeaa65/3402a500-47ed-4144-af75-73ef246582be"
 					(reference "#PWR010")
@@
 		)
 		(instances
-			(project "projet-KiCad"
+			(project "cms-KiCad"
 				(path "/59f7da0b-cec5-4ac9-8c02-026d0daeaa65/3402a500-47ed-4144-af75-73ef246582be"
 					(reference "C10")
@@
 		)
 		(instances
-			(project "projet-KiCad"
+			(project "cms-KiCad"
 				(path "/59f7da0b-cec5-4ac9-8c02-026d0daeaa65/3402a500-47ed-4144-af75-73ef246582be"
 					(reference "#PWR027")
@@
 		)
 		(instances
-			(project "projet-KiCad"
+			(project "cms-KiCad"
 				(path "/59f7da0b-cec5-4ac9-8c02-026d0daeaa65/3402a500-47ed-4144-af75-73ef246582be"
 					(reference "R6")
