File: carteCMS/cms-KiCad/cms-KiCad.kicad_pcb (KiCad board)
At the start: 2 copper layers, 100 x 100 mm, 40 parts, among them IC1 CD4093BM, J1 Conn_01x02, J2 Conn_01x16, J3 AVR-ISP-6, J4 HP, SW1 SW_SPDT, SW2 SW-MCIPTG23K-V, SW3 SW-MCIPTG23K-V, SW4 SW-MCIPTG23K-V, U1 LM358, U3 max7426cua+T, U6 ATmega8U2-A, Y2 Crystal

Commit message: initial - non terminé
Parts:
- moved C8 11.0 mm to (163.2, 86.2), turned to -90 degrees
- moved J3 5.90 mm to (165.8, 82.3), turned to 180 degrees
Routing:
- net /Analog/100xFc: track 15.6 -> 117.6 mm, vias 1 -> 2
- net /Analog/Fmesure: track 14.6 -> 109.3 mm
- net Net-(J2-Pin_10): track 49.3 -> 94.9 mm, vias 0 -> 1
- net Net-(J2-Pin_9): track 65.2 -> 99.5 mm, vias 0 -> 1
- net Net-(J2-Pin_11): track 45.0 -> 75.5 mm
- net Net-(J2-Pin_12): track 41.5 -> 71.5 mm
- net RESET: track 14.5 -> 44.4 mm, vias 0 -> 1
- net Net-(J2-Pin_13): track 38.1 -> 67.6 mm
- net Net-(J2-Pin_14): track 34.6 -> 63.9 mm
- net RS: track 85.7 -> 105.3 mm
- net R/W: track 82.0 -> 100.9 mm
- net E: track 78.3 -> 96.5 mm
- net Net-(J2-Pin_7): track 73.6 -> 91.1 mm
- net Net-(J2-Pin_8): track 69.9 -> 86.7 mm
- net +5V: track 144.3 -> 157.6 mm
- added copper zone on B.Cu, net GND
- added copper zone on F.Cu, net GND
